File: Placa_Serbena/Placa_Serbena.kicad_pcb (KiCad board)
At the start: 2 copper layers, 4 parts

Commit message: Placa
Parts:
- removed the REF** at (67.3, 55.9)
- removed the REF** at (67.3, 36.8)
- added REF**: R_0201_0603Metric, Resistor_SMD:R_0201_0603Metric, F.Cu at (126.2, 100.6)
- added REF**: R_0201_0603Metric, Resistor_SMD:R_0201_0603Metric, F.Cu at (126.2, 95.6)
- added REF**: R_0201_0603Metric, Resistor_SMD:R_0201_0603Metric, F.Cu at (126.2, 103.3)
- added REF**: PinHeader_1x08_P2.54mm_Vertical, Connector_PinHeader_2.54mm:PinHeader_1x08_P2.54mm_Vertical, F.Cu at (116.1, 105.8)
- added REF**: R_0201_0603Metric, Resistor_SMD:R_0201_0603Metric, F.Cu at (120.4, 79.4)
- added REF**: Texas_R-PDSO-G8_EP2.95x4.9mm_Mask2.4x3.1mm, Package_SO:Texas_R-PDSO-G8_EP2.95x4.9mm_Mask2.4x3.1mm, F.Cu at (126.6, 81.9)
- added REF**: R_0201_0603Metric, Resistor_SMD:R_0201_0603Metric, F.Cu at (126.2, 93.1)
- added REF**: R_0201_0603Metric, Resistor_SMD:R_0201_0603Metric, F.Cu at (126.2, 90.6)
- added REF**: R_0201_0603Metric, Resistor_SMD:R_0201_0603Metric, F.Cu at (45.6, 79.4)
- added REF**: R_0201_0603Metric, Resistor_SMD:R_0201_0603Metric, F.Cu at (45.6, 77.1)
- added REF**: R_0201_0603Metric, Resistor_SMD:R_0201_0603Metric, F.Cu at (119.1, 80.9)
- added REF**: R_0201_0603Metric, Resistor_SMD:R_0201_0603Metric, F.Cu at (46.9, 75.6)
- added REF**: Texas_R-PDSO-G8_EP2.95x4.9mm_Mask2.4x3.1mm, Package_SO:Texas_R-PDSO-G8_EP2.95x4.9mm_Mask2.4x3.1mm, F.Cu at (53.2, 78.1)
- added REF**: R_0201_0603Metric, Resistor_SMD:R_0201_0603Metric, F.Cu at (53.8, 85.7)
- added REF**: R_0201_0603Metric, Resistor_SMD:R_0201_0603Metric, F.Cu at (53.8, 88.3)
- added REF**: R_0201_0603Metric, Resistor_SMD:R_0201_0603Metric, F.Cu at (53.8, 90.8)
- added REF**: R_0201_0603Metric, Resistor_SMD:R_0201_0603Metric, F.Cu at (53.8, 93.3)
- added REF**: R_0201_0603Metric, Resistor_SMD:R_0201_0603Metric, F.Cu at (53.8, 95.7)
- added REF**: R_0201_0603Metric, Resistor_SMD:R_0201_0603Metric, F.Cu at (53.8, 98.4)
- added REF**: R_0201_0603Metric, Resistor_SMD:R_0201_0603Metric, F.Cu at (53.8, 83.2)
- added REF**: PinHeader_1x20_P2.54mm_Vertical, Connector_PinHeader_2.54mm:PinHeader_1x20_P2.54mm_Vertical, F.Cu at (67.8, 37.5)
- added REF**: R_0201_0603Metric, Resistor_SMD:R_0201_0603Metric, F.Cu at (126.2, 88.0)
- added REF**: PinHeader_1x08_P2.54mm_Vertical, Connector_PinHeader_2.54mm:PinHeader_1x08_P2.54mm_Vertical, F.Cu at (60.2, 98.4)
- added REF**: PinHeader_1x08_P2.54mm_Vertical, Connector_PinHeader_2.54mm:PinHeader_1x08_P2.54mm_Vertical, F.Cu at (43.7, 101.0)
- added REF**: PinHeader_1x08_P2.54mm_Vertical, Connector_PinHeader_2.54mm:PinHeader_1x08_P2.54mm_Vertical, F.Cu at (51.3, 101.0)
- added REF**: PinHeader_1x14_P2.54mm_Vertical, Connector_PinHeader_2.54mm:PinHeader_1x14_P2.54mm_Vertical, F.Cu at (42.4, 37.5)
- added REF**: R_0201_0603Metric, Resistor_SMD:R_0201_0603Metric, F.Cu at (126.2, 98.2)
- added REF**: PinHeader_1x20_P2.54mm_Vertical, Connector_PinHeader_2.54mm:PinHeader_1x20_P2.54mm_Vertical, F.Cu at (140.8, 37.7)
- added REF**: R_0201_0603Metric, Resistor_SMD:R_0201_0603Metric, F.Cu at (119.1, 83.2)
- added REF**: PinHeader_1x08_P2.54mm_Vertical, Connector_PinHeader_2.54mm:PinHeader_1x08_P2.54mm_Vertical, F.Cu at (123.7, 105.8)
- added REF**: PinHeader_1x14_P2.54mm_Vertical, Connector_PinHeader_2.54mm:PinHeader_1x14_P2.54mm_Vertical, F.Cu at (115.4, 37.7)
- added REF**: PinHeader_1x08_P2.54mm_Vertical, Connector_PinHeader_2.54mm:PinHeader_1x08_P2.54mm_Vertical, F.Cu at (133.2, 98.7)
- moved REF** 114.2 mm to (156.1, 37.7)
- moved REF** 32.3 mm to (83.1, 37.5)
Routing:
- net (no net): track 0.00 -> 874.4 mm
- net GNDREF: track 0.00 -> 156.2 mm
- added copper zone on F.Cu, net GNDREF
Other:
- net class Default: trace_width 0.25 -> 1.5; via_dia 0.8 -> 1.5; via_drill 0.4 -> 1
- net class Mini added: clearance 0.2, trace_width 0.8, via_dia 0.8, via_drill 0.7

Commit message: placa
Parts:
- removed the REF** at (45.6, 77.1)
- removed the REF** at (46.9, 75.6)
- removed the REF** at (53.8, 85.7)
- removed the REF** at (53.8, 90.8)
- removed the REF** at (53.8, 95.7)
- added REF**: R_0201_0603Metric, Resistor_SMD:R_0201_0603Metric, F.Cu at (-44.5, 76.8)
- added REF**: R_0201_0603Metric, Resistor_SMD:R_0201_0603Metric, F.Cu at (-43.2, 75.2)
- added REF**: R_0201_0603Metric, Resistor_SMD:R_0201_0603Metric, F.Cu at (-36.2, 85.3)
- added REF**: R_0201_0603Metric, Resistor_SMD:R_0201_0603Metric, F.Cu at (-36.2, 90.4)
- added REF**: R_0201_0603Metric, Resistor_SMD:R_0201_0603Metric, F.Cu at (-36.2, 95.4)
- moved REF** 90.0 mm to (-44.5, 79.0)
- moved REF** 90.0 mm to (-36.8, 77.7)
- moved REF** 90.0 mm to (-36.2, 87.9)
- moved REF** 90.0 mm to (-36.2, 93.0)
- moved REF** 90.0 mm to (-36.2, 98.0)
- moved REF** 90.0 mm to (-36.2, 82.8)
- moved REF** 90.0 mm to (-22.2, 37.1)
- moved REF** 90.0 mm to (-29.8, 98.0)
- moved REF** 90.0 mm to (-46.4, 100.6)
- moved REF** 90.0 mm to (-38.7, 100.6)
- moved REF** 90.0 mm to (-47.6, 37.1)
- moved REF** 90.0 mm to (-6.99, 37.1)
- moved REF** 89.2 mm to (44.8, 86.7)
- moved REF** 89.2 mm to (37.8, 88.6)
- moved REF** 89.2 mm to (37.8, 83.7)
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