File: Placa_Serbena/Placa_Serbena.kicad_pcb (KiCad board)
At the start: 2 copper layers, 34 parts

Commit message: Amplificador check
Parts:
- removed the REF** at (126.2, 100.6)
- removed the REF** at (126.2, 95.6)
- removed the REF** at (126.2, 103.3)
- removed the REF** at (120.4, 79.4)
- removed the REF** at (126.2, 93.1)
- removed the REF** at (126.2, 90.6)
- removed the REF** at (119.1, 80.9)
- removed the REF** at (126.2, 88.0)
- removed the REF** at (126.2, 98.2)
- removed the REF** at (119.1, 83.2)
- added REF**: R_0805_2012Metric, Resistor_SMD:R_0805_2012Metric, F.Cu at (127.0, 103.4)
- added REF**: R_0805_2012Metric, Resistor_SMD:R_0805_2012Metric, F.Cu at (127.3, 90.7)
- added REF**: R_0805_2012Metric, Resistor_SMD:R_0805_2012Metric, F.Cu at (127.3, 88.1)
- added REF**: R_0805_2012Metric, Resistor_SMD:R_0805_2012Metric, F.Cu at (115.6, 79.0)
- added REF**: R_0805_2012Metric, Resistor_SMD:R_0805_2012Metric, F.Cu at (115.6, 82.3)
- added REF**: R_0805_2012Metric, Resistor_SMD:R_0805_2012Metric, F.Cu at (119.9, 77.7)
- added REF**: R_0805_2012Metric, Resistor_SMD:R_0805_2012Metric, F.Cu at (127.0, 100.6)
- added REF**: R_0805_2012Metric, Resistor_SMD:R_0805_2012Metric, F.Cu at (127.0, 98.3)
- added REF**: R_0805_2012Metric, Resistor_SMD:R_0805_2012Metric, F.Cu at (127.3, 95.5)
- added REF**: R_0805_2012Metric, Resistor_SMD:R_0805_2012Metric, F.Cu at (127.3, 93.0)
Connections:
- REF** pad 1: (no net) -> GNDREF
- REF** pad 4: (no net) -> GNDREF
Routing:
- net (no net): track 874.4 -> 947.0 mm
- net GNDREF: track 156.2 -> 227.4 mm

Commit message: track 07
Parts:
- removed the REF** at (127.3, 90.7)
- removed the REF** at (45.6, 79.4)
- removed the REF** at (45.6, 77.1)
- removed the REF** at (46.9, 75.6)
- removed the REF** at (53.2, 78.1)
- removed the REF** at (53.8, 85.7)
- removed the REF** at (53.8, 88.3)
- removed the REF** at (53.8, 90.8)
- removed the REF** at (53.8, 93.3)
- removed the REF** at (53.8, 95.7)
- removed the REF** at (53.8, 98.4)
- removed the REF** at (53.8, 83.2)
- removed the REF** at (67.8, 37.5)
- removed the REF** at (115.6, 79.0)
- removed the REF** at (60.2, 98.4)
- removed the REF** at (43.7, 101.0)
- removed the REF** at (51.3, 101.0)
- removed the REF** at (42.4, 37.5)
- removed the REF** at (83.1, 37.5)
- removed the REF** at (115.6, 82.3)
- removed the REF** at (127.0, 100.6)
- removed the REF** at (127.0, 98.3)
- removed the REF** at (127.3, 95.5)
- removed the REF** at (127.3, 93.0)
- added REF**: R_0805_2012Metric, Resistor_SMD:R_0805_2012Metric, F.Cu at (35.3, 76.5)
- added REF**: R_0805_2012Metric, Resistor_SMD:R_0805_2012Metric, F.Cu at (23.6, 64.8)
- added REF**: R_0805_2012Metric, Resistor_SMD:R_0805_2012Metric, F.Cu at (23.6, 68.1)
- added REF**: R_0805_2012Metric, Resistor_SMD:R_0805_2012Metric, F.Cu at (35.1, 86.4)
- added REF**: R_0805_2012Metric, Resistor_SMD:R_0805_2012Metric, F.Cu at (35.1, 84.1)
- added REF**: R_0805_2012Metric, Resistor_SMD:R_0805_2012Metric, F.Cu at (35.3, 81.3)
- added REF**: R_0805_2012Metric, Resistor_SMD:R_0805_2012Metric, F.Cu at (35.3, 78.7)
- moved REF** 93.0 mm to (35.1, 89.2)
- moved REF** 93.0 mm to (35.3, 73.9)
- moved REF** 93.0 mm to (41.3, 84.5)
- moved REF** 93.0 mm to (24.1, 91.6)
- moved REF** 93.0 mm to (34.7, 67.7)
- moved REF** 93.0 mm to (27.9, 63.5)
- moved REF** 93.0 mm to (31.8, 91.6)
- moved REF** 93.0 mm to (23.5, 23.5)
- moved REF** 93.0 mm to (64.1, 23.5)
- moved REF** 93.0 mm to (48.9, 23.5)
Routing:
- net (no net): track 947.0 -> 512.6 mm
- net GNDREF: track 227.4 -> 151.2 mm

Commit message: Placa
Parts:
- added REF**: Texas_R-PDSO-G8_EP2.95x4.9mm_Mask2.4x3.1mm, Package_SO:Texas_R-PDSO-G8_EP2.95x4.9mm_Mask2.4x3.1mm, F.Cu at (87.0, 69.3)
