File: Placa_Serbena/Placa_Serbena.sch (KiCad schematic (older format))
At the start: 16 parts

Commit message: Pos testes
Parts:
- removed 100nF: C, symbol Device:C
- removed J?: XLR3_Ground_Switched, symbol Connector:XLR3_Ground_Switched
- removed J?: Conn_01x06_Female, symbol Connector:Conn_01x06_Female
- removed J?: Conn_01x06_Male, symbol Connector:Conn_01x06_Male
- removed U?: STM32F103C8Tx, Package_QFP:LQFP-48_7x7mm_P0.5mm, symbol MCU_ST_STM32F1:STM32F103C8Tx
- added SW?: SW_DPDT_x2, symbol Switch:SW_DPDT_x2
- added U?: stm32f103c8t6-module-china, myelin-kicad:stm32f103c8t6-module-china, symbol stm32f103c8t6-module-china:stm32f103c8t6-module-china
- gave numbers to parts that had none: 11
Connections:
- net +5V: now also U?.18 (5V)
- net GNDREF: now also U2.4 (DGND), U3.4 (DGND), U?.19 (GND)
- net at U2.3 (CAP/2.5V): no longer U3.3 (CAP/2.5V)
- net at U2.5 (MCLK): no longer U3.5 (MCLK)
- net at U2.6 (SDATA), U3.6 (SDATA): now also U?.32 (A7/MOSI1)
- net at U2.7 (SCLK), U3.7 (SCLK): now also U?.30 (A5/SCK1)
- net at U2.8 (~FSYNC): now also U?.33 (B0)
- net at R2.1, U4.1: now also SW?.2 (B)
- net at R6.1, U5.1: now also U?.25 (A0/WKUP)
- net at R4.2: now also SW?.3 (C)
- net at R3.2: now also SW?.1 (A)
- net at U3.10 (VOUT): now also U?.26 (A1)
- net at U3.8 (~FSYNC): now also U?.34 (B1)
Other:
- moved on the sheet: J2, R1, R2, R3, R4, R5, R6, U2, U3, U4A, U5A

Commit message: Segundo amp
Parts:
- removed R5, R6: R, symbol Device:R
- removed U5: LM324, symbol Amplifier_Operational:LM324
- U?: symbol stm32f103c8t6-module-china:stm32f103c8t6-module-china -> Placa_Serbena-rescue:stm32f103c8t6-module-china-stm32f103c8t6-module-china
- renumbered R1 to 100r, R2 to 200r
Changed lines of the file:
@@
 Wire Wire Line
 	6700 2100 7050 2100
-Wire Wire Line
-	8250 2000 8700 2000
 $Comp
 L power:GNDREF #PWR0101
@@
 $EndComp
 $Comp
-L Device:R R2
+L Device:R 200r
 U 1 1 60DF3CBE
 P 6450 2500
-F 0 "R2" V 6243 2500 50  0000 C CNN
+F 0 "200r" V 6243 2500 50  0000 C CNN
 F 1 "R" V 6334 2500 50  0000 C CNN
 F 2 "" V 6380 2500 50  0001 C CNN
@@
 $EndComp
 $Comp
-L Device:R R1
+L Device:R 100r
 U 1 1 60DF477B
 P 6100 2750
-F 0 "R1" H 6170 2796 50  0000 L CNN
+F 0 "100r" H 6170 2796 50  0000 L CNN
 F 1 "R" H 6170 2705 50  0000 L CNN
 F 2 "" V 6030 2750 50  0001 C CNN
@@
 	6100 2900 6100 3000
 Connection ~ 6700 2100
-$Comp
-L Amplifier_Operational:LM324 U5
-U 1 1 60E18353
-P 9000 2100
-F 0 "U5" H 9000 2467 50  0000 C CNN
-F 1 "LM324" H 9000 2376 50  0000 C CNN
-F 2 "" H 8950 2200 50  0001 C CNN
-F 3 "http://www.ti.com/lit/ds/symlink/lm2902-n.pdf" H 9050 2300 50  0001 C CNN
-	1    9000 2100
-	1    0    0    -1
-$EndComp
-$Comp
-L power:GNDREF #PWR0102
-U 1 1 60E1835B
-P 8700 3000
-F 0 "#PWR0102" H 8700 2750 50  0001 C CNN
-F 1 "GNDREF" H 8705 2827 50  0000 C CNN
-F 2 "" H 8700 3000 50  0001 C CNN
-F 3 "" H 8700 3000 50  0001 C CNN
-	1    8700 3000
-	1    0    0    -1
-$EndComp
-$Comp
-L Device:R R6
-U 1 1 60E18361
-P 9050 2500
-F 0 "R6" V 8843 2500 50  0000 C CNN
-F 1 "R" V 8934 2500 50  0000 C CNN
-F 2 "" V 8980 2500 50  0001 C CNN
-F 3 "~" H 9050 2500 50  0001 C CNN
-	1    9050 2500
-	0    1    1    0
-$EndComp
-$Comp
-L Device:R R5
-U 1 1 60E18367
-P 8700 2750
-F 0 "R5" H 8770 2796 50  0000 L CNN
-F 1 "R" H 8770 2705 50  0000 L CNN
-F 2 "" V 8630 2750 50  0001 C CNN
-F 3 "~" H 8700 2750 50  0001 C CNN
-	1    8700 2750
-	1    0    0    -1
-$EndComp
-Wire Wire Line
-	8700 2200 8700 2500
-Wire Wire Line
-	8900 2500 8700 2500
-Connection ~ 8700 2500
-Wire Wire Line
-	8700 2500 8700 2600
-Wire Wire Line
-	9300 2100 9300 2500
-Wire Wire Line
-	9300 2500 9200 2500
-Wire Wire Line
-	8700 2900 8700 3000
 $Comp
 L power:GNDREF #PWR0103
@@
 Wire Wire Line
 	7950 2000 8250 2000
-Connection ~ 8250 2000
 Wire Wire Line
 	8250 2200 8250 2500
@@
 	4900 2000 6100 2000
 Wire Wire Line
-	9300 2100 9550 2100
-Connection ~ 9300 2100
-Wire Wire Line
 	4400 2400 4400 2550
 Wire Wire Line
@@
 	4900 3850 5100 3850
 $Comp
-L stm32f103c8t6-module-china:stm32f103c8t6-module-china U?
+L Placa_Serbena-rescue:stm32f103c8t6-module-china-stm32f103c8t6-module-china U?
 U 1 1 61304A6A
 P 2050 2800
@@
 Wire Wire Line
 	3200 4900 9550 4900
-Wire Wire Line
-	9550 4900 9550 2100
 $Comp
 L Switch:SW_DPDT_x2 SW?
